File: devices/lune-v6/hardware/heatvalve-6-rev2.1/heatvalve-6-rev2.1.kicad_sch (KiCad schematic)
At the start: 128 parts, among them J1 USB4105-GF-A, J10 ONEWIRE 3, J11 I2C EXPANSION DNP, J2 MOTOR 1 4P4C, J3 MOTOR 2 4P4C, J4 MOTOR 3 4P4C, J5 MOTOR 4 4P4C, J6 MOTOR 5 4P4C, J7 MOTOR 6 4P4C, J8 ONEWIRE 1, J9 ONEWIRE 2, SW1 RESET, SW2 BOOT, U1 ESP32-S3-WROOM-1-N16R8, U10 MCP6004, U11 LM339B, U12 74HC74, U13 74HC4051, U14 74HC4051, U2 USBLC6-2SC6, U21 DRV8837DSGR, U22 DRV8837DSGR, U23 DRV8837DSGR, U24 DRV8837DSGR, U25 DRV8837DSGR, U26 DRV8837DSGR, U3 MT2492, U9 INA180A1 (x20)

Commit message: Regenerate Lune V6 rev2 hardware design
Parts:
- removed C32, C34, C36, C38, C40, C50, C51: 100n, Capacitor_SMD:C_0603_1608Metric, symbol Device:C
- removed C33, C35, C37, C39, C41: 1u, Capacitor_SMD:C_0805_2012Metric, symbol Device:C
- removed R78, R79, R80, R81: 10k, Resistor_SMD:R_0603_1608Metric, symbol Device:R
- removed U13, U14: 74HC4051, Package_SO:TSSOP-16_4.4x5mm_P0.65mm, symbol 74xx:74HC4051
- removed U22, U23, U24, U25, U26: DRV8837DSGR, Package_SON:WSON-8-1EP_2x2mm_P0.5mm_EP0.9x1.6mm, symbol Driver_Motor:DRV8837
- added U31: LOW_RON_BILATERAL_SPST MUX 1, Package_TO_SOT_SMD:SOT-23-6, symbol Connector_Generic:Conn_01x06
- added U32: LOW_RON_BILATERAL_SPST MUX 2, Package_TO_SOT_SMD:SOT-23-6, symbol Connector_Generic:Conn_01x06
- added U33: LOW_RON_BILATERAL_SPST MUX 3, Package_TO_SOT_SMD:SOT-23-6, symbol Connector_Generic:Conn_01x06
- added U34: LOW_RON_BILATERAL_SPST MUX 4, Package_TO_SOT_SMD:SOT-23-6, symbol Connector_Generic:Conn_01x06
- added U35: LOW_RON_BILATERAL_SPST MUX 5, Package_TO_SOT_SMD:SOT-23-6, symbol Connector_Generic:Conn_01x06
- added U36: LOW_RON_BILATERAL_SPST MUX 6, Package_TO_SOT_SMD:SOT-23-6, symbol Connector_Generic:Conn_01x06
- R60, R61: value 100k -> 10k
- R62: value 100k -> 1M
- R70, R71, R72, R73, R74, R75, R76, R77: value 10k -> 100k
- U21: value DRV8837DSGR -> DRV8837DSGR shared H-bridge
Connections:
- net BEMF_A1 is gone; now on net GND: R70.2
- net BEMF_A2 is gone; now on net GND: R72.2
- net BEMF_A3 is gone; now on net GND: R74.2
- net BEMF_A4 is gone; now on net GND: R76.2
- net BEMF_B1 is gone; now on net GND: R71.2
- net BEMF_B2 is gone; now on net GND: R73.2
- net BEMF_B3 is gone; now on net GND: R75.2
- net BEMF_B4 is gone; now on net GND: R77.2
- net MOT5_A is gone; now on net MOT_COM: J6.2 (Pin_2)
- net MOT6_A is gone; now on net MOT_COM: J7.2 (Pin_2)
- net PH2 is gone; now on net MUX_EN5: U1.18 (IO10)
- net PH4 is gone; now on net HBR_IN1: U1.20 (IO12)
- net +3V3_SYS: now also U31.1 (Pin_1), U32.1 (Pin_1), U33.1 (Pin_1), U34.1 (Pin_1), U35.1 (Pin_1), U36.1 (Pin_1)
- net BEMF_MUX_A: now also R60.2
- net BEMF_MUX_B: now also R61.2
- net GND: now also U31.2 (Pin_2), U32.2 (Pin_2), U33.2 (Pin_2), U34.2 (Pin_2), U35.2 (Pin_2), U36.2 (Pin_2); no longer R60.2, R61.2
- net BEMF_SEL0 renamed MOT_COM
- net MOT_COM: now also J2.2 (Pin_2), J3.2 (Pin_2), J4.2 (Pin_2), J5.2 (Pin_2), U21.2 (OUT1); no longer U1.6 (IO6)
- net BEMF_SEL1 renamed MOT_DRV
- net MOT_DRV: now also R62.1, U21.3 (OUT2), U31.4 (Pin_4), U32.4 (Pin_4), U33.4 (Pin_4), U34.4 (Pin_4), U35.4 (Pin_4), U36.4 (Pin_4); no longer U1.7 (IO7)
- net BEMF_SEL2 renamed MUX_EN3
- net MUX_EN3: now also R74.1, U33.3 (Pin_3); no longer R62.1
- net EN1: no longer names the net of U1.24 (IO47)
- net EN1: no longer U21.5 (IN2)
- net EN2: no longer names the net of U1.25 (IO48)
- net EN3: no longer names the net of U1.31 (IO38)
- net EN4: no longer names the net of U1.32 (IO39)
- net EN5: no longer names the net of U1.33 (IO40)
- net EN6: no longer names the net of U1.34 (IO41)
- removed net MOT1_A: J2.2 (Pin_2), R70.1, U21.2 (OUT1)
- removed net MOT1_B: J2.3 (Pin_3), R71.1, U21.3 (OUT2)
- net MOT2_A renamed MUX_EN1
- net MUX_EN1: now also U1.6 (IO6), U31.3 (Pin_3); no longer J3.2 (Pin_2)
- net MOT2_B renamed MOT2_SEL
- net MOT2_SEL: now also U32.5 (Pin_5); no longer R73.1
- removed net MOT3_A: J4.2 (Pin_2), R74.1
- net MOT3_B renamed MOT3_SEL
- net MOT3_SEL: now also U33.5 (Pin_5); no longer R75.1
- net MOT4_A renamed MUX_EN5
- net MUX_EN5: now also U35.3 (Pin_3); no longer J5.2 (Pin_2)
- net MOT4_B renamed MOT4_SEL
- net MOT4_SEL: now also U34.5 (Pin_5); no longer R77.1
- net MOT5_B renamed MOT5_SEL
- net MOT5_SEL: now also U35.5 (Pin_5)
- net MOT6_B renamed MOT6_SEL
- net MOT6_SEL: now also U36.5 (Pin_5)
- net PH1 renamed HBR_IN1
- net HBR_IN1: now also R70.1; no longer U1.17 (IO9)
- net PH3 renamed MUX_EN6
- net MUX_EN6: now also R77.1, U36.3 (Pin_3)
- net PH5 renamed HBR_IN2
- net HBR_IN2: now also R71.1, U21.5 (IN2)
- net PH6: no longer names the net of U1.22 (IO14)
- new net MOT1_SEL: J2.3 (Pin_3), U31.5 (Pin_5)
- new net MUX_EN2: R73.1, U1.7 (IO7), U32.3 (Pin_3)
- new net MUX_EN4: R75.1, U1.17 (IO9), U34.3 (Pin_3)
- no-connect marks 27 -> 40
Other:
- note added: "30mA=0.60V, 60mA=1.20V, 150mA=3.00V. Current is endstop/load/force evidence."
- note added: "Connector pinout: 1 NC, 2 shared MOT_COM, 3 selected MOTx_SEL, 4 NC."
- note added: "Firmware and hardware review must guarantee exactly one MUX_EN active during drive."
- note added: "Only one mux channel may be enabled; the selected motor is visible on MOT_COM/MOT_DRV."
- note added: "SHARED DRV8837 + 6 x MOTOR MUX / 4P4C OUTPUTS"
- note added: "SHARED MOTOR BUS BEMF / TACHO"
- note added: "TACHO_EDGE is the required commutation-count channel; ADC_BEMF qualifies it."
- note added: "USB-C VBUS is the only board power input; +3V3_SYS powers logic and motors."
- note removed: "30mA=0.60V, 60mA=1.20V, 150mA=3.00V. Engagement current remains measurable."
- note removed: "6 x DRV8837 / 4P4C MOTOR OUTPUTS"
- note removed: "ADC_BEMF is differential motion evidence; TACHO_EDGE counts qualified commutation."
- note removed: "Connector pinout: 1 NC, 2 MOT_A, 3 MOT_B, 4 NC (center pair)."
- note removed: "SELECTED DIFFERENTIAL BEMF / TACHO"
