File: lune-v6/hardware/lune-v6-rev3.2/lune-v6-rev3.2-analog.kicad_sch (KiCad schematic)
At the start: 43 parts, among them Q1 2N7002 ARM INHIBIT, Q2 2N7002 TIMEOUT FAULT, U32 INA180A1 x20, U34 LMV393, U35 74LVC1G74DP,125, U36 74HC4060D,653, U37 TLV9001IDBVR

Commit message: Add placement floorplan SVG and geometry JSON for Lune V6 rev3.2
- Introduced a new SVG file for the component placement floorplan, detailing the layout and dimensions of the Lune V6 rev3.2 hardware.
- Added a JSON file containing the geometric coordinates for each component, including reference designators and their respective positions on the board.
Parts:
- removed C24: 100n, Capacitor_SMD:C_0603_1608Metric, symbol Device:C
- removed C25: 22n 5% 50V C0G, Capacitor_SMD:C_1206_3216Metric, symbol Device:C
- removed Q2: 2N7002 TIMEOUT FAULT, Package_TO_SOT_SMD:SOT-23, symbol Transistor_FET:2N7002
- removed R27: 180k 1%, Resistor_SMD:R_0603_1608Metric, symbol Device:R
- removed R28: 360k 1%, Resistor_SMD:R_0603_1608Metric, symbol Device:R
- removed U36: 74HC4060D,653, Package_SO:SOIC-16_3.9x9.9mm_P1.27mm, symbol 74xx:74HC4060
Connections:
- no-connect marks 9 -> 0
Other:
- note added: "Hysteresis (R49/R50) is on the comparator non-inverting input."
- note added: "No hardware max-on-time: the firmware runtime limit and tacho stall evidence bound actuator travel. See actuator_overrun_hazard."
- note removed: "4060 Q14 with 180k/360k/22n C0G: 71.4 s typical; release only after 50..90 s characterization and Rt trim."
- note removed: "Hysteresis (R49/R50) is on the comparator non-inverting input. 4060 MR = LATCH_STATE bounds total ARMED time."
