File: lune-v6/hardware/lune-v6-rev3.2/lune-v6-rev3.2-power.kicad_sch (KiCad schematic)
At the start: 23 parts, among them J1 TYPE-C-31-M-12, U2 TPS2553DBVR-1, U3 SY8089AAAC, U4 AP2112K-3.3TRG1, U5 USBLC6-2SC6

Commit message: Refactor code structure for improved readability and maintainability
Parts:
- C10, C2, C4, C7: value 10u 10V -> 10u 16V; footprint Capacitor_SMD:C_0805_2012Metric -> Capacitor_SMD:C_0603_1608Metric; Dielectric (none) -> X5R_RATIFIED_VERIFY_EFFECTIVE_C_AT_3V3; LCSC C380346 -> C18164635; MPN TCC0805X7R106K100FT -> TCC0603X5R106K160CT
- FB1: footprint Inductor_SMD:L_0603_1608Metric_Pad1.05x0.95mm_HandSolder -> Inductor_SMD:L_0603_1608Metric
